File: KiCad/adorobo_kitagami.kicad_pcb (KiCad board)
At the start: 2 copper layers, 80 x 60 mm, 71 parts, among them IC1 TC4051BP, J1 USB_C_Receptacle_USB2.0_16P, J10 Conn_01x02, J2 Conn_01x15_Socket, J3 PWR IN, J5 Conn_01x15_Socket, J6 Conn_01x06, J9 Conn_01x02, SW1 SW_Push, SW2 SW_Push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

Commit message: I have documented the changes made.
Parts:
- renumbered D6 to D4
Changed lines of the file:
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@@
     (property "ki_keywords" "LED diode light-emitting-diode")
     (attr smd)
-    (fp_text reference "D6" (at -2.875 0) (layer "F.SilkS" knockout)
+    (fp_text reference "D4" (at -2.875 0) (layer "F.SilkS" knockout)
         (effects (font (size 1 1) (thickness 0.15)))
     )
